File: MicroTetra887.kicad_pcb (KiCad board)
At the start: 2 copper layers, 16 parts, among them J1 USB_B, J11 VGA DE15, J14 Conn_01x06, J15 Conn_01x06, SW11 SW_Push, U2 74LS161, Y2 CXO_DIP8

Commit message: Add files via upload
Parts:
- removed R2: R_US, Resistor_THT:R_Axial_DIN0207_L6.3mm_D2.5mm_P10.16mm_Horizontal
- removed RN1, RN2: R_Network08_US, Resistor_THT:R_Array_SIP9
- removed U2: 74LS161, Package_DIP:DIP-16_W7.62mm_Socket
- removed Y2: CXO_DIP8, Oscillator:Oscillator_DIP-8
- added C1: C_Polarized_US, Capacitor_THT:CP_Radial_Tantal_D6.0mm_P2.50mm, F.Cu at (98.7, 107.5)
- added C2: C_Polarized_US, Capacitor_THT:CP_Radial_Tantal_D6.0mm_P2.50mm, F.Cu at (116.3, 107.5)
- added C3: C_Polarized_US, Capacitor_THT:CP_Radial_D8.0mm_P3.50mm, F.Cu at (122.5, 68.3)
- added C4: C_Polarized_US, Capacitor_THT:CP_Radial_D8.0mm_P3.50mm, F.Cu at (85.0, 105.8)
- added C5: C_Polarized_US, Capacitor_THT:CP_Radial_D8.0mm_P3.50mm, F.Cu at (132.5, 68.3)
- added C8: C_Small, Capacitor_THT:C_Disc_D3.8mm_W2.6mm_P2.50mm, F.Cu at (101.2, 101.2)
- added C9: C_Small, Capacitor_THT:C_Disc_D3.8mm_W2.6mm_P2.50mm, F.Cu at (96.2, 78.8)
- added G100: LOGO, MicroTetra887:Logo, B.Cu at (90.0, 87.5)
- added G101: LOGO, MicroTetra887:Title, F.Cu at (135.0, 93.8)
- added J16: Conn_01x06, Connector_PinSocket_2.54mm:PinSocket_1x06_P2.54mm_Horizontal, F.Cu at (145.0, 98.0)
- added J8: DB9_Male, Connector_Dsub:DSUB-9_Pins_Horizontal_P2.77x2.84mm_EdgePinOffset7.70mm_Housed_MountingHolesOffset9.12mm, F.Cu at (74.5, 138.2)
- added J9: DB9_Male, Connector_Dsub:DSUB-9_Pins_Horizontal_P2.77x2.84mm_EdgePinOffset7.70mm_Housed_MountingHolesOffset9.12mm, F.Cu at (114.5, 138.2)
- added JP1: SolderJumper_2_Open, Jumper:SolderJumper-2_P1.3mm_Open_Pad1.0x1.5mm, B.Cu at (78.8, 132.5)
- added JP10: SolderJumper_2_Open, Jumper:SolderJumper-2_P1.3mm_Open_Pad1.0x1.5mm, B.Cu at (112.5, 132.5)
- added JP11: SolderJumper_2_Open, Jumper:SolderJumper-2_P1.3mm_Open_Pad1.0x1.5mm, B.Cu at (116.2, 132.5)
- added JP12: SolderJumper_2_Open, Jumper:SolderJumper-2_P1.3mm_Open_Pad1.0x1.5mm, B.Cu at (120.0, 132.5)
- added JP2: SolderJumper_2_Open, Jumper:SolderJumper-2_P1.3mm_Open_Pad1.0x1.5mm, B.Cu at (82.5, 132.5)
- added JP3: SolderJumper_2_Open, Jumper:SolderJumper-2_P1.3mm_Open_Pad1.0x1.5mm, B.Cu at (86.2, 132.5)
- added JP4: SolderJumper_2_Open, Jumper:SolderJumper-2_P1.3mm_Open_Pad1.0x1.5mm, B.Cu at (90.0, 132.5)
- added JP5: SolderJumper_2_Open, Jumper:SolderJumper-2_P1.3mm_Open_Pad1.0x1.5mm, B.Cu at (93.8, 132.5)
- added JP6: SolderJumper_2_Open, Jumper:SolderJumper-2_P1.3mm_Open_Pad1.0x1.5mm, B.Cu at (97.5, 132.5)
- added JP7: SolderJumper_2_Open, Jumper:SolderJumper-2_P1.3mm_Open_Pad1.0x1.5mm, B.Cu at (101.2, 132.5)
- added JP8: SolderJumper_2_Open, Jumper:SolderJumper-2_P1.3mm_Open_Pad1.0x1.5mm, B.Cu at (105.0, 132.5)
- added JP9: SolderJumper_2_Open, Jumper:SolderJumper-2_P1.3mm_Open_Pad1.0x1.5mm, B.Cu at (108.8, 132.5)
- added R11: R_US, Resistor_THT:R_Axial_DIN0207_L6.3mm_D2.5mm_P10.16mm_Horizontal, F.Cu at (112.6, 60.0)
- added R18: R_US, Resistor_THT:R_Axial_DIN0207_L6.3mm_D2.5mm_P10.16mm_Horizontal, F.Cu at (75.0, 117.4)
- added R19: R_US, Resistor_THT:R_Axial_DIN0207_L6.3mm_D2.5mm_P10.16mm_Horizontal, F.Cu at (78.8, 117.4)
- added R20: R_US, Resistor_THT:R_Axial_DIN0207_L6.3mm_D2.5mm_P10.16mm_Horizontal, F.Cu at (82.5, 117.4)
- added R21: R_US, Resistor_THT:R_Axial_DIN0207_L6.3mm_D2.5mm_P10.16mm_Horizontal, F.Cu at (86.2, 117.4)
- added R22: R_US, Resistor_THT:R_Axial_DIN0207_L6.3mm_D2.5mm_P10.16mm_Horizontal, F.Cu at (90.0, 117.4)
- added R23: R_US, Resistor_THT:R_Axial_DIN0207_L6.3mm_D2.5mm_P10.16mm_Horizontal, F.Cu at (93.8, 117.4)
- added R24: R_US, Resistor_THT:R_Axial_DIN0207_L6.3mm_D2.5mm_P10.16mm_Horizontal, F.Cu at (97.5, 117.4)
- added R25: R_US, Resistor_THT:R_Axial_DIN0207_L6.3mm_D2.5mm_P10.16mm_Horizontal, F.Cu at (101.2, 117.4)
- added R26: R_US, Resistor_THT:R_Axial_DIN0207_L6.3mm_D2.5mm_P10.16mm_Horizontal, F.Cu at (105.0, 117.4)
- added R27: R_US, Resistor_THT:R_Axial_DIN0207_L6.3mm_D2.5mm_P10.16mm_Horizontal, F.Cu at (108.8, 117.4)
- added R28: R_US, Resistor_THT:R_Axial_DIN0207_L6.3mm_D2.5mm_P10.16mm_Horizontal, F.Cu at (112.5, 117.4)
- added R29: R_US, Resistor_THT:R_Axial_DIN0207_L6.3mm_D2.5mm_P10.16mm_Horizontal, F.Cu at (116.2, 117.4)
- added R30: R_US, Resistor_THT:R_Axial_DIN0207_L6.3mm_D2.5mm_P10.16mm_Horizontal, F.Cu at (120.0, 117.4)
- added SW1: SW_Push, Button_Switch_THT:SW_PUSH_6mm_H13mm, F.Cu at (134.2, 127.8)
- added SW2: SW_Push, Button_Switch_THT:SW_PUSH_6mm_H13mm, F.Cu at (134.2, 112.2)
- added SW3: SW_Push, Button_Switch_THT:SW_PUSH_6mm_H13mm, F.Cu at (142.0, 120.0)
- added SW4: SW_Push, Button_Switch_THT:SW_PUSH_6mm_H13mm, F.Cu at (126.5, 120.0)
- added SW5: SW_Push, Button_Switch_THT:SW_PUSH_6mm_H13mm, F.Cu at (62.5, 120.0)
- added SW6: SW_Push, Button_Switch_THT:SW_PUSH_6mm_H13mm, F.Cu at (51.5, 120.0)
- added TP1: TestPoint, MicroTetra887:ScrewHole-4-40, F.Cu at (54.0, 54.0)
- added TP10: TestPoint, MicroTetra887:PinHeader_1x01_P2.54mm_Vertical_TestPoint, F.Cu at (51.4, 91.4)
- added TP100: TestPoint, MicroTetra887:PinHeader_1x01_P2.54mm_Vertical_TestPoint, F.Cu at (59.1, 116.8)
- added TP101: TestPoint, MicroTetra887:PinHeader_1x01_P2.54mm_Vertical_TestPoint, F.Cu at (61.6, 99.1)
- added TP102: TestPoint, MicroTetra887:PinHeader_1x01_P2.54mm_Vertical_TestPoint, F.Cu at (61.6, 101.6)
- added TP103: TestPoint, MicroTetra887:PinHeader_1x01_P2.54mm_Vertical_TestPoint, F.Cu at (61.6, 104.1)
- added TP104: TestPoint, MicroTetra887:PinHeader_1x01_P2.54mm_Vertical_TestPoint, F.Cu at (61.6, 106.7)
- added TP105: TestPoint, MicroTetra887:PinHeader_1x01_P2.54mm_Vertical_TestPoint, F.Cu at (61.6, 109.2)
- added TP106: TestPoint, MicroTetra887:PinHeader_1x01_P2.54mm_Vertical_TestPoint, F.Cu at (61.6, 111.8)
- added TP107: TestPoint, MicroTetra887:PinHeader_1x01_P2.54mm_Vertical_TestPoint, F.Cu at (61.6, 114.3)
- added TP108: TestPoint, MicroTetra887:PinHeader_1x01_P2.54mm_Vertical_TestPoint, F.Cu at (61.6, 116.8)
- added TP109: TestPoint, MicroTetra887:PinHeader_1x01_P2.54mm_Vertical_TestPoint, F.Cu at (64.1, 99.1)
- added TP11: TestPoint, MicroTetra887:PinHeader_1x01_P2.54mm_Vertical_TestPoint, F.Cu at (51.4, 94.0)
- added TP110: TestPoint, MicroTetra887:PinHeader_1x01_P2.54mm_Vertical_TestPoint, F.Cu at (64.1, 101.6)
- added TP111: TestPoint, MicroTetra887:PinHeader_1x01_P2.54mm_Vertical_TestPoint, F.Cu at (64.1, 104.1)
- added TP112: TestPoint, MicroTetra887:PinHeader_1x01_P2.54mm_Vertical_TestPoint, F.Cu at (64.1, 106.7)
- added TP113: TestPoint, MicroTetra887:PinHeader_1x01_P2.54mm_Vertical_TestPoint, F.Cu at (64.1, 109.2)
- added TP114: TestPoint, MicroTetra887:PinHeader_1x01_P2.54mm_Vertical_TestPoint, F.Cu at (64.1, 111.8)
- added TP115: TestPoint, MicroTetra887:PinHeader_1x01_P2.54mm_Vertical_TestPoint, F.Cu at (64.1, 114.3)
- added TP116: TestPoint, MicroTetra887:PinHeader_1x01_P2.54mm_Vertical_TestPoint, F.Cu at (64.1, 116.8)
- added TP117: TestPoint, MicroTetra887:PinHeader_1x01_P2.54mm_Vertical_TestPoint, F.Cu at (66.7, 99.1)
- added TP118: TestPoint, MicroTetra887:PinHeader_1x01_P2.54mm_Vertical_TestPoint, F.Cu at (66.7, 101.6)
- added TP119: TestPoint, MicroTetra887:PinHeader_1x01_P2.54mm_Vertical_TestPoint, F.Cu at (66.7, 104.1)
- added TP12: TestPoint, MicroTetra887:PinHeader_1x01_P2.54mm_Vertical_TestPoint, F.Cu at (51.4, 96.5)
- added TP120: TestPoint, MicroTetra887:PinHeader_1x01_P2.54mm_Vertical_TestPoint, F.Cu at (66.7, 106.7)
- added TP121: TestPoint, MicroTetra887:PinHeader_1x01_P2.54mm_Vertical_TestPoint, F.Cu at (66.7, 109.2)
- added TP122: TestPoint, MicroTetra887:PinHeader_1x01_P2.54mm_Vertical_TestPoint, F.Cu at (66.7, 111.8)
- added TP123: TestPoint, MicroTetra887:PinHeader_1x01_P2.54mm_Vertical_TestPoint, F.Cu at (66.7, 114.3)
- added TP124: TestPoint, MicroTetra887:PinHeader_1x01_P2.54mm_Vertical_TestPoint, F.Cu at (66.7, 116.8)
- added TP125: TestPoint, MicroTetra887:PinHeader_1x01_P2.54mm_Vertical_TestPoint, F.Cu at (69.2, 99.1)
- added TP126: TestPoint, MicroTetra887:PinHeader_1x01_P2.54mm_Vertical_TestPoint, F.Cu at (69.2, 101.6)
- added TP127: TestPoint, MicroTetra887:PinHeader_1x01_P2.54mm_Vertical_TestPoint, F.Cu at (69.2, 104.1)
- added TP128: TestPoint, MicroTetra887:PinHeader_1x01_P2.54mm_Vertical_TestPoint, F.Cu at (69.2, 106.7)
- added TP129: TestPoint, MicroTetra887:PinHeader_1x01_P2.54mm_Vertical_TestPoint, F.Cu at (69.2, 109.2)
- added TP13: TestPoint, MicroTetra887:PinHeader_1x01_P2.54mm_Vertical_TestPoint, F.Cu at (54.0, 78.7)
- added TP130: TestPoint, MicroTetra887:PinHeader_1x01_P2.54mm_Vertical_TestPoint, F.Cu at (69.2, 111.8)
- added TP131: TestPoint, MicroTetra887:PinHeader_1x01_P2.54mm_Vertical_TestPoint, F.Cu at (69.2, 114.3)
- added TP132: TestPoint, MicroTetra887:PinHeader_1x01_P2.54mm_Vertical_TestPoint, F.Cu at (69.2, 116.8)
- added TP14: TestPoint, MicroTetra887:PinHeader_1x01_P2.54mm_Vertical_TestPoint, F.Cu at (54.0, 81.3)
- added TP15: TestPoint, MicroTetra887:PinHeader_1x01_P2.54mm_Vertical_TestPoint, F.Cu at (54.0, 83.8)
- added TP16: TestPoint, MicroTetra887:PinHeader_1x01_P2.54mm_Vertical_TestPoint, F.Cu at (54.0, 86.4)
- added TP17: TestPoint, MicroTetra887:PinHeader_1x01_P2.54mm_Vertical_TestPoint, F.Cu at (54.0, 88.9)
- added TP18: TestPoint, MicroTetra887:PinHeader_1x01_P2.54mm_Vertical_TestPoint, F.Cu at (54.0, 91.4)
- added TP19: TestPoint, MicroTetra887:PinHeader_1x01_P2.54mm_Vertical_TestPoint, F.Cu at (54.0, 94.0)
- added TP2: TestPoint, MicroTetra887:ScrewHole-4-40, F.Cu at (146.0, 54.0)
- added TP20: TestPoint, MicroTetra887:PinHeader_1x01_P2.54mm_Vertical_TestPoint, F.Cu at (54.0, 96.5)
- added TP21: TestPoint, MicroTetra887:PinHeader_1x01_P2.54mm_Vertical_TestPoint, F.Cu at (56.5, 78.7)
- added TP22: TestPoint, MicroTetra887:PinHeader_1x01_P2.54mm_Vertical_TestPoint, F.Cu at (56.5, 81.3)
- added TP23: TestPoint, MicroTetra887:PinHeader_1x01_P2.54mm_Vertical_TestPoint, F.Cu at (56.5, 83.8)
- added TP24: TestPoint, MicroTetra887:PinHeader_1x01_P2.54mm_Vertical_TestPoint, F.Cu at (56.5, 86.4)
- added TP25: TestPoint, MicroTetra887:PinHeader_1x01_P2.54mm_Vertical_TestPoint, F.Cu at (56.5, 88.9)
- added TP26: TestPoint, MicroTetra887:PinHeader_1x01_P2.54mm_Vertical_TestPoint, F.Cu at (56.5, 91.4)
- added TP27: TestPoint, MicroTetra887:PinHeader_1x01_P2.54mm_Vertical_TestPoint, F.Cu at (56.5, 94.0)
- added TP28: TestPoint, MicroTetra887:PinHeader_1x01_P2.54mm_Vertical_TestPoint, F.Cu at (56.5, 96.5)
- added TP29: TestPoint, MicroTetra887:PinHeader_1x01_P2.54mm_Vertical_TestPoint, F.Cu at (59.1, 78.7)
- added TP3: TestPoint, MicroTetra887:ScrewHole-4-40, F.Cu at (146.0, 146.0)
- added TP30: TestPoint, MicroTetra887:PinHeader_1x01_P2.54mm_Vertical_TestPoint, F.Cu at (59.1, 81.3)
- added TP31: TestPoint, MicroTetra887:PinHeader_1x01_P2.54mm_Vertical_TestPoint, F.Cu at (59.1, 83.8)
- added TP32: TestPoint, MicroTetra887:PinHeader_1x01_P2.54mm_Vertical_TestPoint, F.Cu at (59.1, 86.4)
- added TP33: TestPoint, MicroTetra887:PinHeader_1x01_P2.54mm_Vertical_TestPoint, F.Cu at (59.1, 88.9)
- added TP34: TestPoint, MicroTetra887:PinHeader_1x01_P2.54mm_Vertical_TestPoint, F.Cu at (59.1, 91.4)
- added TP35: TestPoint, MicroTetra887:PinHeader_1x01_P2.54mm_Vertical_TestPoint, F.Cu at (59.1, 94.0)
- added TP36: TestPoint, MicroTetra887:PinHeader_1x01_P2.54mm_Vertical_TestPoint, F.Cu at (59.1, 96.5)
- added TP37: TestPoint, MicroTetra887:PinHeader_1x01_P2.54mm_Vertical_TestPoint, F.Cu at (61.6, 78.7)
- added TP38: TestPoint, MicroTetra887:PinHeader_1x01_P2.54mm_Vertical_TestPoint, F.Cu at (61.6, 81.3)
- added TP39: TestPoint, MicroTetra887:PinHeader_1x01_P2.54mm_Vertical_TestPoint, F.Cu at (61.6, 83.8)
- added TP4: TestPoint, MicroTetra887:ScrewHole-4-40, F.Cu at (54.0, 146.0)
- added TP40: TestPoint, MicroTetra887:PinHeader_1x01_P2.54mm_Vertical_TestPoint, F.Cu at (61.6, 86.4)
- added TP41: TestPoint, MicroTetra887:PinHeader_1x01_P2.54mm_Vertical_TestPoint, F.Cu at (61.6, 88.9)
- added TP42: TestPoint, MicroTetra887:PinHeader_1x01_P2.54mm_Vertical_TestPoint, F.Cu at (61.6, 91.4)
- added TP43: TestPoint, MicroTetra887:PinHeader_1x01_P2.54mm_Vertical_TestPoint, F.Cu at (61.6, 94.0)
- added TP44: TestPoint, MicroTetra887:PinHeader_1x01_P2.54mm_Vertical_TestPoint, F.Cu at (61.6, 96.5)
- added TP45: TestPoint, MicroTetra887:PinHeader_1x01_P2.54mm_Vertical_TestPoint, F.Cu at (64.1, 78.7)
- added TP46: TestPoint, MicroTetra887:PinHeader_1x01_P2.54mm_Vertical_TestPoint, F.Cu at (64.1, 81.3)
- added TP47: TestPoint, MicroTetra887:PinHeader_1x01_P2.54mm_Vertical_TestPoint, F.Cu at (64.1, 83.8)
- added TP48: TestPoint, MicroTetra887:PinHeader_1x01_P2.54mm_Vertical_TestPoint, F.Cu at (64.1, 86.4)
- added TP49: TestPoint, MicroTetra887:PinHeader_1x01_P2.54mm_Vertical_TestPoint, F.Cu at (64.1, 88.9)
- added TP5: TestPoint, MicroTetra887:PinHeader_1x01_P2.54mm_Vertical_TestPoint, F.Cu at (51.4, 78.7)
- added TP50: TestPoint, MicroTetra887:PinHeader_1x01_P2.54mm_Vertical_TestPoint, F.Cu at (64.1, 91.4)
- added TP51: TestPoint, MicroTetra887:PinHeader_1x01_P2.54mm_Vertical_TestPoint, F.Cu at (64.1, 94.0)
- added TP52: TestPoint, MicroTetra887:PinHeader_1x01_P2.54mm_Vertical_TestPoint, F.Cu at (64.1, 96.5)
- added TP53: TestPoint, MicroTetra887:PinHeader_1x01_P2.54mm_Vertical_TestPoint, F.Cu at (66.7, 78.7)
- added TP54: TestPoint, MicroTetra887:PinHeader_1x01_P2.54mm_Vertical_TestPoint, F.Cu at (66.7, 81.3)
- added TP55: TestPoint, MicroTetra887:PinHeader_1x01_P2.54mm_Vertical_TestPoint, F.Cu at (66.7, 83.8)
- added TP56: TestPoint, MicroTetra887:PinHeader_1x01_P2.54mm_Vertical_TestPoint, F.Cu at (66.7, 86.4)
- added TP57: TestPoint, MicroTetra887:PinHeader_1x01_P2.54mm_Vertical_TestPoint, F.Cu at (66.7, 88.9)
- added TP58: TestPoint, MicroTetra887:PinHeader_1x01_P2.54mm_Vertical_TestPoint, F.Cu at (66.7, 91.4)
- added TP59: TestPoint, MicroTetra887:PinHeader_1x01_P2.54mm_Vertical_TestPoint, F.Cu at (66.7, 94.0)
- added TP6: TestPoint, MicroTetra887:PinHeader_1x01_P2.54mm_Vertical_TestPoint, F.Cu at (51.4, 81.3)
- added TP60: TestPoint, MicroTetra887:PinHeader_1x01_P2.54mm_Vertical_TestPoint, F.Cu at (66.7, 96.5)
- added TP61: TestPoint, MicroTetra887:PinHeader_1x01_P2.54mm_Vertical_TestPoint, F.Cu at (69.2, 78.7)
- added TP62: TestPoint, MicroTetra887:PinHeader_1x01_P2.54mm_Vertical_TestPoint, F.Cu at (69.2, 81.3)
- added TP63: TestPoint, MicroTetra887:PinHeader_1x01_P2.54mm_Vertical_TestPoint, F.Cu at (69.2, 83.8)
- added TP64: TestPoint, MicroTetra887:PinHeader_1x01_P2.54mm_Vertical_TestPoint, F.Cu at (69.2, 86.4)
- added TP65: TestPoint, MicroTetra887:PinHeader_1x01_P2.54mm_Vertical_TestPoint, F.Cu at (69.2, 88.9)
- added TP66: TestPoint, MicroTetra887:PinHeader_1x01_P2.54mm_Vertical_TestPoint, F.Cu at (69.2, 91.4)
- added TP67: TestPoint, MicroTetra887:PinHeader_1x01_P2.54mm_Vertical_TestPoint, F.Cu at (69.2, 94.0)
- added TP68: TestPoint, MicroTetra887:PinHeader_1x01_P2.54mm_Vertical_TestPoint, F.Cu at (69.2, 96.5)
- added TP69: TestPoint, MicroTetra887:PinHeader_1x01_P2.54mm_Vertical_TestPoint, F.Cu at (51.4, 99.1)
- added TP7: TestPoint, MicroTetra887:PinHeader_1x01_P2.54mm_Vertical_TestPoint, F.Cu at (51.4, 83.8)
- added TP70: TestPoint, MicroTetra887:PinHeader_1x01_P2.54mm_Vertical_TestPoint, F.Cu at (51.4, 101.6)
- added TP71: TestPoint, MicroTetra887:PinHeader_1x01_P2.54mm_Vertical_TestPoint, F.Cu at (51.4, 104.1)
- added TP72: TestPoint, MicroTetra887:PinHeader_1x01_P2.54mm_Vertical_TestPoint, F.Cu at (51.4, 106.7)
- added TP73: TestPoint, MicroTetra887:PinHeader_1x01_P2.54mm_Vertical_TestPoint, F.Cu at (51.4, 109.2)
- added TP74: TestPoint, MicroTetra887:PinHeader_1x01_P2.54mm_Vertical_TestPoint, F.Cu at (51.4, 111.8)
- added TP75: TestPoint, MicroTetra887:PinHeader_1x01_P2.54mm_Vertical_TestPoint, F.Cu at (51.4, 114.3)
- added TP76: TestPoint, MicroTetra887:PinHeader_1x01_P2.54mm_Vertical_TestPoint, F.Cu at (51.4, 116.8)
- added TP77: TestPoint, MicroTetra887:PinHeader_1x01_P2.54mm_Vertical_TestPoint, F.Cu at (54.0, 99.1)
- added TP78: TestPoint, MicroTetra887:PinHeader_1x01_P2.54mm_Vertical_TestPoint, F.Cu at (54.0, 101.6)
- added TP79: TestPoint, MicroTetra887:PinHeader_1x01_P2.54mm_Vertical_TestPoint, F.Cu at (54.0, 104.1)
- added TP8: TestPoint, MicroTetra887:PinHeader_1x01_P2.54mm_Vertical_TestPoint, F.Cu at (51.4, 86.4)
- added TP80: TestPoint, MicroTetra887:PinHeader_1x01_P2.54mm_Vertical_TestPoint, F.Cu at (54.0, 106.7)
- added TP81: TestPoint, MicroTetra887:PinHeader_1x01_P2.54mm_Vertical_TestPoint, F.Cu at (54.0, 109.2)
- added TP82: TestPoint, MicroTetra887:PinHeader_1x01_P2.54mm_Vertical_TestPoint, F.Cu at (54.0, 111.8)
- added TP83: TestPoint, MicroTetra887:PinHeader_1x01_P2.54mm_Vertical_TestPoint, F.Cu at (54.0, 114.3)
- added TP84: TestPoint, MicroTetra887:PinHeader_1x01_P2.54mm_Vertical_TestPoint, F.Cu at (54.0, 116.8)
- added TP85: TestPoint, MicroTetra887:PinHeader_1x01_P2.54mm_Vertical_TestPoint, F.Cu at (56.5, 99.1)
- added TP86: TestPoint, MicroTetra887:PinHeader_1x01_P2.54mm_Vertical_TestPoint, F.Cu at (56.5, 101.6)
- added TP87: TestPoint, MicroTetra887:PinHeader_1x01_P2.54mm_Vertical_TestPoint, F.Cu at (56.5, 104.1)
- added TP88: TestPoint, MicroTetra887:PinHeader_1x01_P2.54mm_Vertical_TestPoint, F.Cu at (56.5, 106.7)
- added TP89: TestPoint, MicroTetra887:PinHeader_1x01_P2.54mm_Vertical_TestPoint, F.Cu at (56.5, 109.2)
- added TP9: TestPoint, MicroTetra887:PinHeader_1x01_P2.54mm_Vertical_TestPoint, F.Cu at (51.4, 88.9)
- added TP90: TestPoint, MicroTetra887:PinHeader_1x01_P2.54mm_Vertical_TestPoint, F.Cu at (56.5, 111.8)
- added TP91: TestPoint, MicroTetra887:PinHeader_1x01_P2.54mm_Vertical_TestPoint, F.Cu at (56.5, 114.3)
- added TP92: TestPoint, MicroTetra887:PinHeader_1x01_P2.54mm_Vertical_TestPoint, F.Cu at (56.5, 116.8)
- added TP93: TestPoint, MicroTetra887:PinHeader_1x01_P2.54mm_Vertical_TestPoint, F.Cu at (59.1, 99.1)
- added TP94: TestPoint, MicroTetra887:PinHeader_1x01_P2.54mm_Vertical_TestPoint, F.Cu at (59.1, 101.6)
- added TP95: TestPoint, MicroTetra887:PinHeader_1x01_P2.54mm_Vertical_TestPoint, F.Cu at (59.1, 104.1)
- added TP96: TestPoint, MicroTetra887:PinHeader_1x01_P2.54mm_Vertical_TestPoint, F.Cu at (59.1, 106.7)
- added TP97: TestPoint, MicroTetra887:PinHeader_1x01_P2.54mm_Vertical_TestPoint, F.Cu at (59.1, 109.2)
- added TP98: TestPoint, MicroTetra887:PinHeader_1x01_P2.54mm_Vertical_TestPoint, F.Cu at (59.1, 111.8)
- added TP99: TestPoint, MicroTetra887:PinHeader_1x01_P2.54mm_Vertical_TestPoint, F.Cu at (59.1, 114.3)
- added U1: PIC16F887-IP, Package_DIP:DIP-40_W15.24mm_Socket, F.Cu at (75.9, 97.6)
- added Y1: Crystal, Crystal:Crystal_HC18-U_Vertical, F.Cu at (105.0, 107.5)
- moved SW11 69.8 mm to (105.2, 52.7)
- moved J14 62.5 mm to (55.0, 62.5)
- moved R17 57.5 mm to (105.3, 70.0), turned to 180 degrees
- moved R16 50.4 mm to (105.3, 73.8), turned to 180 degrees
- moved R15 41.8 mm to (90.3, 73.8), turned to 180 degrees
- moved R14 41.5 mm to (90.3, 70.0), turned to 180 degrees
- moved J15 35.1 mm to (145.0, 75.2), turned to 180 degrees
- moved R10 33.9 mm to (75.2, 73.8), turned to 180 degrees
- moved R9 33.7 mm to (75.2, 70.0), turned to 180 degrees
- moved J11 28.7 mm to (75.7, 64.8), turned to 180 degrees
- moved J1 22.0 mm to (126.0, 60.3), turned to 90 degrees
Connections:
- J14 pad 2: +3V3 -> +5V
- R17 pad 1: unconnected-(R17-Pad1) -> VGA-BLUE-OUT
Routing:
- net ~{MCLR}: track 0.00 -> 100.1 mm, vias 0 -> 1
- net JOY-SELECT: track 0.00 -> 93.6 mm, vias 0 -> 1
- net JOY2-BUTTON2: track 0.00 -> 78.9 mm
- net JOY2-RIGHT: track 0.00 -> 76.5 mm, vias 0 -> 2
- net BTN-BUTTON2: track 0.00 -> 75.9 mm, vias 0 -> 2
- net JOY2-BUTTON1: track 0.00 -> 74.7 mm, vias 0 -> 1
- net BTN-DOWN: track 0.00 -> 73.9 mm, vias 0 -> 3
- net JOY2-LEFT: track 0.00 -> 73.4 mm, vias 0 -> 2
- net JOY2-DOWN: track 0.00 -> 71.6 mm, vias 0 -> 2
- net BTN-LEFT: track 0.00 -> 70.6 mm, vias 0 -> 2
- net JOY2-UP: track 0.00 -> 69.8 mm
- net BTN-UP: track 0.00 -> 65.5 mm, vias 0 -> 2
- net JOY1-BUTTON1: track 0.00 -> 63.1 mm
- net BTN-BUTTON1: track 0.00 -> 63.0 mm, vias 0 -> 3
- net VGA-H-SYNC: track 0.00 -> 58.3 mm
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- added copper zone on In2.Cu, net +5V
- added copper zone on In1.Cu, net GND
Other:
- board outline added: 100 x 100 mm
- copper layers 2 -> 4
- board text added: "*"
- board text added: "- TX RX - - GND"
- board text added: "BUTTONS-TO-JOY1 ----"
- board text added: "BUTTONS-TO-JOY2 ----"
- board text added: "GND +5V MISO MOSI CLK CS"
- board text added: "MCLR +5V GND DAT CLK -"
- board text added: "Professor Steven Chad Burrow stevenchadburrow@gmail.com github.com/stevenchadburrow youtube.com/user/stevenchadburrow August 2026"
