File: MicroTetra887.kicad_pcb (KiCad board)
At the start: 4 copper layers, 100 x 100 mm, 189 parts, among them J1 USB_B, J11 VGA DE15, J14 Conn_01x06, J15 Conn_01x06, J16 Conn_01x06, J8 DB9_Male, J9 DB9_Male, SW1 SW_Push, SW11 SW_Push, SW2 SW_Push, SW3 SW_Push, SW4 SW_Push, SW5 SW_Push, SW6 SW_Push, U1 PIC16F887-IP, Y1 Crystal

Commit message: Add files via upload
Parts:
- added SW7: SW_SPDT, Button_Switch_THT:SW_E-Switch_EG1224_SPDT_Angled, F.Cu at (136.5, 57.8)
- moved R11 46.1 mm to (73.8, 84.9), turned to -90 degrees
- moved JP1 15.0 mm to (78.8, 117.5), turned to -90 degrees
- moved JP10 15.0 mm to (112.5, 117.5), turned to -90 degrees
- moved JP11 15.0 mm to (116.2, 117.5), turned to -90 degrees
- moved JP12 15.0 mm to (120.0, 117.5), turned to -90 degrees
- moved JP2 15.0 mm to (82.5, 117.5), turned to -90 degrees
- moved JP3 15.0 mm to (86.2, 117.5), turned to -90 degrees
- moved JP4 15.0 mm to (90.0, 117.5), turned to -90 degrees
- moved JP5 15.0 mm to (93.8, 117.5), turned to -90 degrees
- moved JP6 15.0 mm to (97.5, 117.5), turned to -90 degrees
- moved JP7 15.0 mm to (101.2, 117.5), turned to -90 degrees
- moved JP8 15.0 mm to (105.0, 117.5), turned to -90 degrees
- moved JP9 15.0 mm to (108.8, 117.5), turned to -90 degrees
- moved J1 12.2 mm to (113.8, 60.3)
- moved SW11 7.50 mm to (97.7, 52.7)
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Connections:
- J1 pad 1: +5V -> POWER
Routing:
- net POWER: track 0.00 -> 25.9 mm
- net BTN-DOWN: track 73.9 -> 62.9 mm, vias 3 -> 2
- net JOY2-RIGHT: track 76.5 -> 86.8 mm, vias 2 -> 0
- net VGA-INT-PIX: track 51.5 -> 57.5 mm
- net BTN-RIGHT: track 54.5 -> 48.8 mm
- net JOY2-UP: track 69.8 -> 75.3 mm
- net BTN-LEFT: track 70.6 -> 65.2 mm
- net VGA-GREEN-PIX: track 28.8 -> 33.9 mm, vias 1 -> 0
- net VGA-BLUE-PIX: track 14.8 -> 19.8 mm
- net VGA-RED-PIX: track 41.4 -> 46.5 mm, vias 1 -> 0
- net +5V: track 27.6 -> 32.5 mm
- net BTN-BUTTON1: track 63.0 -> 58.5 mm, vias 3 -> 2
- net JOY1-BUTTON1: track 63.1 -> 58.8 mm
- net JOY-SELECT: track 93.6 -> 97.9 mm
- net VGA-V-SYNC: track 51.0 -> 55.2 mm
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Other:
- outline, holes or cut-outs redrawn
