File: MicroTetra887.kicad_sch (KiCad schematic)
At the start: 20 parts, among them J1 USB_B, J11 VGA DE15, J14 Conn_01x06, J15 Conn_01x06, J8 DB9_Male, J9 DB9_Male, SW11 SW_Push, U1 PIC16F887-IP, Y1 Crystal

Commit message: Add files via upload
Parts:
- removed R2: R_US, Resistor_THT:R_Axial_DIN0207_L6.3mm_D2.5mm_P10.16mm_Horizontal, symbol Device:R_US
- removed RN1, RN2: R_Network08_US, Resistor_THT:R_Array_SIP9, symbol Device:R_Network08_US
- added C3, C4, C5: C_Polarized_US, Capacitor_THT:CP_Radial_D8.0mm_P3.50mm, symbol Device:C_Polarized_US
- added C8, C9: C_Small, Capacitor_THT:C_Disc_D3.8mm_W2.6mm_P2.50mm, symbol Device:C_Small
- added J16: Conn_01x06, Connector_PinSocket_2.54mm:PinSocket_1x06_P2.54mm_Horizontal, symbol Connector_Generic:Conn_01x06
- added JP1, JP10, JP11, JP12, JP2, JP3, JP4, JP5, JP6, JP7, JP8, JP9: SolderJumper_2_Open, Jumper:SolderJumper-2_P1.3mm_Open_Pad1.0x1.5mm, symbol Jumper:SolderJumper_2_Open
- added R11, R18, R19, R20, R21, R22, R23, R24, R25, R26, R27, R28, R29, R30: R_US, Resistor_THT:R_Axial_DIN0207_L6.3mm_D2.5mm_P10.16mm_Horizontal, symbol Device:R_US
- added SW1, SW2, SW3, SW4, SW5, SW6: SW_Push, Button_Switch_THT:SW_PUSH_6mm_H13mm, symbol Switch:SW_Push
- added TP1, TP2, TP3, TP4: TestPoint, MicroTetra887:ScrewHole-4-40, symbol Connector:TestPoint
- added TP10, TP100, TP101, TP102, TP103, TP104, TP105, TP106, TP107, TP108, TP109, TP11, TP110, TP111, TP112, TP113, TP114, TP115, TP116, TP117, TP118, TP119, TP12, TP120, TP121, TP122, TP123, TP124, TP125, TP126, TP127, TP128, TP129, TP13, TP130, TP131, TP132, TP14, TP15, TP16, TP17, TP18, TP19, TP20, TP21, TP22, TP23, TP24, TP25, TP26, TP27, TP28, TP29, TP30, TP31, TP32, TP33, TP34, TP35, TP36, TP37, TP38, TP39, TP40, TP41, TP42, TP43, TP44, TP45, TP46, TP47, TP48, TP49, TP5, TP50, TP51, TP52, TP53, TP54, TP55, TP56, TP57, TP58, TP59, TP6, TP60, TP61, TP62, TP63, TP64, TP65, TP66, TP67, TP68, TP69, TP7, TP70, TP71, TP72, TP73, TP74, TP75, TP76, TP77, TP78, TP79, TP8, TP80, TP81, TP82, TP83, TP84, TP85, TP86, TP87, TP88, TP89, TP9, TP90, TP91, TP92, TP93, TP94, TP95, TP96, TP97, TP98, TP99: TestPoint, MicroTetra887:PinHeader_1x01_P2.54mm_Vertical_TestPoint, symbol Connector:TestPoint
- C1: footprint (none) -> Capacitor_THT:CP_Radial_Tantal_D6.0mm_P2.50mm; Field5 (none) -> 22pF
- C2: footprint (none) -> Capacitor_THT:CP_Radial_Tantal_D6.0mm_P2.50mm
- J14: Field4 ICSP for PICkit/SNAP -> ICSP for PICkit
- J8, J9: footprint Library:DSUB-9-custom_Male_Horizontal_P2.77x2.84mm_EdgePinOffset7.70mm_Housed_MountingHolesOffset9.12mm -> Connector_Dsub:DSUB-9_Pins_Horizontal_P2.77x2.84mm_EdgePinOffset7.70mm_Housed_MountingHolesOffset9.12mm
- U1: footprint (none) -> Package_DIP:DIP-40_W15.24mm_Socket
- Y1: footprint (none) -> Crystal:Crystal_HC18-U_Vertical
Connections:
- net +3V3 is gone; now on net +5V: J14.2 (Pin_2)
- net +5V: now also C3.1, C4.1, C5.1, C8.1, C9.1, J16.5 (Pin_5), R11.1, R18.1, R19.1, R20.1, R21.1, R22.1, R23.1, R24.1, R25.1, R26.1, R27.1, R28.1, R29.1, R30.1
- net GND: now also C3.2, C4.2, C5.2, C8.2, C9.2, J16.6 (Pin_6), SW1.2, SW2.2, SW3.2, SW4.2, SW5.2, SW6.2, TP1.1, TP2.1, TP3.1, TP4.1
- net JOY-SELECT: now also U1.8 (RE0/AN5), R18.2; no longer U1.15 (T10S0/T1CKI/RC0)
- net JOY1-BUTTON1: now also JP5.2 (B), R23.2
- net JOY1-BUTTON2: now also JP6.2 (B), R24.2
- net JOY1-DOWN: now also JP2.2 (B), R20.2
- net JOY1-LEFT: now also JP3.2 (B), R21.2
- net JOY1-RIGHT: now also JP4.2 (B), R22.2
- net JOY1-UP: now also JP1.2 (B), R19.2
- net JOY2-BUTTON1: now also JP11.2 (B), R29.2
- net JOY2-BUTTON2: now also JP12.2 (B), R30.2
- net JOY2-DOWN: now also JP8.2 (B), R26.2
- net JOY2-LEFT: now also JP9.2 (B), R27.2
- net JOY2-RIGHT: now also JP10.2 (B), R28.2
- net JOY2-UP: now also JP7.2 (B), R25.2
- net VGA-BLUE-OUT: now also R17.1
- net ~{MCLR}: now also R11.2
- net SPI-CLK: now reaches U1.18 (SCL/SCK/RC3)
- net SPI-CLK: now also J16.2 (Pin_2)
- net SPI-MISO: now reaches U1.23 (SDA/SDI/RC4)
- net SPI-MISO: now also J16.4 (Pin_4)
- net SPI-MOSI: now reaches U1.24 (SDO/RC5)
- net SPI-MOSI: now also J16.3 (Pin_3)
- new net BTN-BUTTON1: JP11.1 (A), JP5.1 (A), SW5.1
- new net BTN-BUTTON2: JP12.1 (A), JP6.1 (A), SW6.1
- new net BTN-DOWN: JP2.1 (A), JP8.1 (A), SW2.1
- new net BTN-LEFT: JP3.1 (A), JP9.1 (A), SW3.1
- new net BTN-RIGHT: JP10.1 (A), JP4.1 (A), SW4.1
- new net BTN-UP: JP1.1 (A), JP7.1 (A), SW1.1
- new net SPI-CS: J16.1 (Pin_1), U1.15 (T10S0/T1CKI/RC0)
- no-connect marks 11 -> 145
Other:
- note added: "680/1.2K ohms"
- note added: "https://falstad.com/circuit/circuitjs.html?ctz=DwYwlgTgBAZgvAIgIwKgFwM6IAwDpsEECsqYIiSeATAVQOx0DM2AHFQGwCcndqIARoiLZUAB0EIALI1QA3CENQBbTEICmAWiQoAfACgoUYAGUoADwrtGVKDRZQkRRu1utU8BCKgAbMDlRoABaIVAgA9PqGJuaW1rYs9o7O8Szu-j5+ngHBCKERBkYASjHIknQ2SJwVZRVUqbDpAO4eXkoAhmayivlRjSVINQ5VDk4ulaENyOGRRn0WpeVD1Yv0Ey3TBcBzFIOrI8mraVM9s-27iwOLjERr-idbZ1c3+y7Xt8czwADmZ0QuVYlJH8oJx2F51vdtqVgZJ2JIHEDXixJEcRJCzgkoMx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"
- note removed: "??? ohms"

Commit message: Add files via upload
Parts:
- added SW7: SW_SPDT, Button_Switch_THT:SW_E-Switch_EG1224_SPDT_Angled, symbol Switch:SW_SPDT
Connections:
- net +5V: now also SW7.2 (B); no longer J1.1 (VBUS)
- new net POWER: J1.1 (VBUS), SW7.1 (A)
- no-connect marks 145 -> 146
